File: Hardware/Xenium2019/Xenium2019.kicad_pcb (KiCad board)
At the start: 2 copper layers, 39.4 x 36.4 mm, 21 parts, among them J1 SM10B-SRSS-TB, Q1 310mA/60V/1.6Ω, Q2 310mA/60V/1.6Ω, Q3 310mA/60V/1.6Ω, Q4 310mA/60V/1.6Ω, U1 XC9572XL-10VQG64, U2 AM29LV160M

Commit message: Panel v1
Parts:
- added G***: LOGO, Xenium2019:board_bottom_logos, B.Cu at (148.7, 105.1)
- moved G*** 0.22 mm to (148.7, 105.2)
Other:
- board text removed: "https://github.com/Ryzee119/OpenXenium"
